Commit message: init

File: aubo_description/urdf/aubo_i3.urdf (robot description, URDF)
Before this commit: robot aubo_i3, 8 links, 7 joints
Joints:
- removed joint foreArm_Joint
- removed joint shoulder_Joint
- removed joint upperArm_Joint
- removed joint wrist1_Joint
- removed joint wrist2_Joint
- removed joint wrist3_Joint
- added joint foreArm_joint: type revolute, parent upperArm_Link, child foreArm_Link, origin xyz=0.266 0 0 rpy=3.1416 0 0, axis 0 0 1, limit lower=-3.05 upper=3.05 effort=0 velocity=0
- added joint shoulder_joint: type revolute, parent base_link, child shoulder_Link, origin xyz=0 0 0.157 rpy=0 0 3.1416, axis 0 0 1, limit lower=-3.05 upper=3.05 effort=0 velocity=0
- added joint upperArm_joint: type revolute, parent shoulder_Link, child upperArm_Link, origin xyz=0 0.119 0 rpy=-1.5708 -1.5708 0, axis 0 0 1, limit lower=-3.05 upper=3.05 effort=0 velocity=0
- added joint wrist1_joint: type revolute, parent foreArm_Link, child wrist1_Link, origin xyz=0.2565 0 0 rpy=3.1416 0 1.5708, axis 0 0 -1, limit lower=-3.05 upper=3.05 effort=0 velocity=0
- added joint wrist2_joint: type revolute, parent wrist1_Link, child wrist2_Link, origin xyz=0 0.1025 0 rpy=-1.5708 0 0, axis 0 0 1, limit lower=-3.05 upper=3.05 effort=0 velocity=0
- added joint wrist3_joint: type revolute, parent wrist2_Link, child wrist3_Link, origin xyz=0 -0.094 0 rpy=1.5708 0 0, axis 0 0 -1, limit lower=-3.05 upper=3.05 effort=0 velocity=0
